File: eagle/max21100_v2.brd (EAGLE design)
At the start: 15.6 x 15.6 mm, 12 parts

Commit message: Improved V2
Parts:
- removed SJ1: SEPARATE VDDIO, max21100:SJ_2S-TRACE
- removed U$2: (no value), ohw-logo:OSHW_8X200_NOTEXT
- added ADDR: (no value), max21100:SJ_3
- added I2C: SOLDERJUMPERNO, max21100:SJ_2S-NO
- added VDDIO: (no value), max21100:SJ_2S-TRACE
- moved R3 1.31 mm to (5.71, 14.1)
- moved LED1 0.85 mm to (9.53, 14.1)
- moved C3 0.32 mm to (8.10, 11.4)
- moved C2 0.16 mm to (9.84, 11.4)
Connections:
- net CS: now also I2C.2
- net DSYNC: now also JP2.2; no longer JP2.4
- net GND: now also ADDR.1
- net INT1: now also JP2.3; no longer JP2.2
- net INT2: now also JP2.4; no longer JP2.3
- net SA0_SDO: now also ADDR.2
- net VDD: now also VDDIO.1; no longer SJ1.1
- net VDDIO: now also ADDR.3, I2C.1, VDDIO.2; no longer SJ1.2
Routing:
- net CS: track 9.72 -> 16.8 mm
- net VDDIO: track 13.4 -> 18.6 mm, vias 0 -> 1
- net MST_SCL: track 9.60 -> 14.0 mm
- net SA0_SDO: track 7.61 -> 11.0 mm
- net MST_SDA: track 12.8 -> 14.6 mm
- net VDD: track 16.8 -> 18.5 mm
- net INT1: track 6.97 -> 5.53 mm
- net GND: track 28.1 -> 27.1 mm, vias 1 -> 2
- net SDA_CLK: track 8.59 -> 9.56 mm
- net INT2: track 5.95 -> 5.11 mm
- net SDA_SDI: track 11.2 -> 11.8 mm
- net DSYNC: track 6.32 -> 6.48 mm, vias 1 -> 0
- removed copper zone on layer 1, net GND
- removed copper zone on layer 16, net GND
Other:
- board text added: "+"
- board text added: "-"
- board text added: "0"
- board text added: "1"
- board text added: "CS"
- board text added: "SA0"
- board text added: "Technical Toys"
- board text removed: "CX=0.1uF"
- board text removed: "R1,R2=4K2"
- board text removed: "R3=360R"
- board text removed: "SDI"
- board text removed: "SDO"
- board text removed: "Technical Toys 2014"
